File: LEDboard.brd (EAGLE design)
At the start: 72 x 72 mm, 285 parts

Commit message: Placed Everything
Parts:
- removed U$1, U$2: IS31FL3741_QFN60, MRRobotBadge:QFN60
- added U1, U2: IS31FL3741_QFN60, MRRobotBadge:QFN60
- moved R43 198.8 mm to (14.6, 26.2), flipped to the bottom, turned to 119.1 degrees
- moved R44 197.2 mm to (16.6, 25.0), flipped to the bottom, turned to 123.6 degrees
- moved R49 196.7 mm to (24.9, 16.7), flipped to the bottom, turned to 146.2 degrees
- moved R45 195.4 mm to (18.5, 23.6), flipped to the bottom, turned to 128.1 degrees
- moved R37 195.1 mm to (1.05, 30.0), flipped to the bottom, turned to 92 degrees
- moved R38 194.7 mm to (3.40, 29.8), flipped to the bottom, turned to 96.5 degrees
- moved R50 194.1 mm to (26.2, 14.7), flipped to the bottom, turned to 150.6 degrees
- moved R39 194.1 mm to (5.74, 29.4), flipped to the bottom, turned to 101 degrees
- moved R46 193.5 mm to (20.3, 22.1), flipped to the bottom, turned to 132.6 degrees
- moved R40 193.3 mm to (8.04, 28.9), flipped to the bottom, turned to 105.6 degrees
- moved R41 192.3 mm to (10.3, 28.2), flipped to the bottom, turned to 110 degrees
- moved R47 191.4 mm to (22.0, 20.4), flipped to the bottom, turned to 137.1 degrees
- moved R51 191.3 mm to (27.2, 12.6), flipped to the bottom, turned to 155.2 degrees
- moved R42 191.2 mm to (12.5, 27.3), flipped to the bottom, turned to 114.6 degrees
- moved R55 189.7 mm to (29.8, 3.52), flipped to the bottom, turned to 173.2 degrees
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Connections:
- net N$1: now also U1.6; no longer U$1.6
- net N$10: now also U1.57; no longer U$1.57
- net N$11: now also U1.56; no longer U$1.56
- net N$12: now also U1.54; no longer U$1.54
- net N$13: now also U2.6; no longer U$2.6
- net N$14: now also U2.5; no longer U$2.5
- net N$15: now also U2.4; no longer U$2.4
- net N$16: now also U1.53; no longer U$1.53
- net N$17: now also U1.52; no longer U$1.52
- net N$18: now also U1.51; no longer U$1.51
- net N$19: now also U2.3; no longer U$2.3
- net N$2: now also U1.5; no longer U$1.5
- net N$20: now also U2.2; no longer U$2.2
- net N$21: now also U2.1; no longer U$2.1
- net N$22: now also U1.50; no longer U$1.50
- net N$23: now also U1.49; no longer U$1.49
- net N$24: now also U1.48; no longer U$1.48
- net N$25: now also U2.60; no longer U$2.60
- net N$26: now also U2.59; no longer U$2.59
- net N$27: now also U2.58; no longer U$2.58
- net N$28: now also U1.47; no longer U$1.47
- net N$29: now also U1.46; no longer U$1.46
- net N$3: now also U1.4; no longer U$1.4
- net N$30: now also U1.45; no longer U$1.45
- net N$31: now also U2.57; no longer U$2.57
- net N$32: now also U2.56; no longer U$2.56
- net N$33: now also U2.54; no longer U$2.54
- net N$34: now also U1.44; no longer U$1.44
- net N$35: now also U1.43; no longer U$1.43
- net N$36: now also U1.42; no longer U$1.42
- net N$37: now also U2.53; no longer U$2.53
- net N$38: now also U2.52; no longer U$2.52
- net N$39: now also U2.51; no longer U$2.51
- net N$4: now also U1.3; no longer U$1.3
- net N$40: now also U1.41; no longer U$1.41
- net N$41: now also U1.40; no longer U$1.40
- net N$42: now also U1.39; no longer U$1.39
- net N$43: now also U2.50; no longer U$2.50
- net N$44: now also U2.49; no longer U$2.49
- net N$45: now also U2.48; no longer U$2.48
- net N$46: now also U1.38; no longer U$1.38
- net N$47: now also U1.37; no longer U$1.37
- net N$48: now also U1.35; no longer U$1.35
- net N$49: now also U2.47; no longer U$2.47
- net N$5: now also U1.2; no longer U$1.2
- net N$50: now also U2.46; no longer U$2.46
- net N$51: now also U2.45; no longer U$2.45
- net N$52: now also U1.34; no longer U$1.34
- net N$53: now also U1.33; no longer U$1.33
- net N$54: now also U1.32; no longer U$1.32
- net N$55: now also U2.44; no longer U$2.44
- net N$56: now also U2.43; no longer U$2.43
- net N$57: now also U2.42; no longer U$2.42
- net N$58: now also U1.31; no longer U$1.31
- net N$59: now also U1.30; no longer U$1.30
- net N$6: now also U1.1; no longer U$1.1
- net N$60: now also U1.29; no longer U$1.29
- net N$61: now also U2.41; no longer U$2.41
- net N$62: now also U2.40; no longer U$2.40
- net N$63: now also U2.39; no longer U$2.39
- net N$64: now also U2.38; no longer U$2.38
- net N$65: now also U2.37; no longer U$2.37
- net N$66: now also U2.35; no longer U$2.35
- net N$67: now also U2.34; no longer U$2.34
- net N$68: now also U2.33; no longer U$2.33
- net N$69: now also U2.32; no longer U$2.32
- net N$7: now also U1.60; no longer U$1.60
- net N$70: now also U2.31; no longer U$2.31
- net N$71: now also U2.30; no longer U$2.30
- net N$72: now also U2.29; no longer U$2.29
- net N$8: now also U1.59; no longer U$1.59
- net N$9: now also U1.58; no longer U$1.58
- net U1SW1: now also U1.16; no longer U$1.16
- net U1SW2: now also U1.17; no longer U$1.17
- net U1SW3: now also U1.18; no longer U$1.18
- net U1SW4: now also U1.19; no longer U$1.19
- net U1SW5: now also U1.20; no longer U$1.20
- net U1SW6: now also U1.21; no longer U$1.21
- net U1SW7: now also U1.22; no longer U$1.22
- net U1SW8: now also U1.23; no longer U$1.23
- net U1SW9: now also U1.24; no longer U$1.24
- net U2SW1: now also U2.16; no longer U$2.16
- net U2SW2: now also U2.17; no longer U$2.17
- net U2SW3: now also U2.18; no longer U$2.18
- net U2SW4: now also U2.19; no longer U$2.19
- net U2SW5: now also U2.20; no longer U$2.20
- net U2SW6: now also U2.21; no longer U$2.21
- net U2SW7: now also U2.22; no longer U$2.22
- net U2SW8: now also U2.23; no longer U$2.23
- net U2SW9: now also U2.24; no longer U$2.24
Other:
- board text removed: "1"
- board text removed: "4"

Commit message: Added more stuff
Parts:
- added B1: 1.8-5V, microbuilder:JSTPH2
- added C1: 10uF, microbuilder:0805-NO
- added C2: 2.2uF, microbuilder:0805-NO
- added C4: 0.1uF, microbuilder:0805-NO
- added C5: 100uF/6V, microbuilder:EIA3528-21/B-R
- added C6: 10µF, microbuilder:0805-NO
- added IC1: REG1117, burr-brown:SOT223
- added J2: (no value), SparkFun-Connectors:USB-B-MICRO-SMD
- added L1: VLC5045-6.8uH, microbuilder:INDUCTOR_5X5MM_TDK_VLC5045
- added LBO: RED, microbuilder:CHIPLED_0805_NOOUTLINE
- added LED3: ORANGE, microbuilder:CHIPLED_0805_NOOUTLINE
- added LED4: GREEN, microbuilder:CHIPLED_0805_NOOUTLINE
- added PWR: BLUE, microbuilder:CHIPLED_0805_NOOUTLINE
- added Q1: MMUN2133LT1G, transistor:SC59-BEC
- added R77, R83, R85: 1K, microbuilder:0805-NO
- added R78, R81: 340K, microbuilder:0805-NO
- added R79, R82: 1.87Mohm, microbuilder:0805-NO
- added R80: 200K, microbuilder:0805-NO
- added R84: 470, microbuilder:0805-NO
- added R86: 2k, microbuilder:0805-NO
- added U3: ATSAMD21G-A, SparkFun-IC-Microcontroller:TQFP-48
- added U4: TPS61090RSAR, microbuilder:PVQFN-16
- added U5: MCP73831T-2ACI/OT, microbuilder:SOT23-5
Connections:
- new net 3V3: IC1.2
- new net 5.0V: C2.1, C5.+, IC1.3, PWR.A, R79.2, U4.1, U4.15, U4.16
- new net ENABLE: R78.2, U4.11
- new net GND: B1.1, C1.2, C2.2, C4.2, C5.-, C6.2, IC1.1, J2.GND, LBO.C, LED4.C, R77.2, R80.1, R81.1, R86.2, U4.10, U4.13, U4.5, U4.6, U4.7, U4.P$18, U4.P$19, U4.P$20, U4.P$21, U4.P$22, U4.THERMAL, U5.2
- new net LBO: Q1.B, U4.12
- new net N$73: L1.P$2, U4.3, U4.4
- new net N$74: R81.2, R82.1, U4.9
- new net N$75: PWR.C, R77.1
- new net N$76: R79.1, R80.2, U4.14
- new net N$77: LBO.A, R83.1
- new net N$78: Q1.C, R83.2
- new net N$79: LED3.C, R84.1
- new net N$80: R84.2, R85.2, U5.1
- new net N$81: R86.1, U5.5
- new net N$82: LED4.A, R85.1
- new net VBAT: B1.2, C1.1, C4.1, L1.P$1, Q1.E, R78.1, R82.2, U4.8, U5.3
- new net VDD1: C6.1, J2.VBUS, LED3.A, U5.4
Routing:
- net VDD1: track 0.00 -> 4.26 mm
- net GND: track 0.00 -> 4.26 mm
- net N$82: track 0.00 -> 1.92 mm
- net N$79: track 0.00 -> 1.92 mm
Other:
- board text added: "CHRG"
- board text added: "DONE"
- board text added: "LOW"

Commit message: placed power
Parts:
- removed C1: 10uF, microbuilder:0805-NO
- removed C4: 0.1uF, microbuilder:0805-NO
- removed R78: 340K, microbuilder:0805-NO
- B1: value 1.8-5V -> S2B-PH-SM4-TB(LF)(SN)
- moved C2 61.5 mm to (0.00, 6.00), flipped to the bottom
- moved R80 60.3 mm to (-3.75, 3.00), flipped to the bottom, turned to 270 degrees
- moved IC1 55.0 mm to (0.00, 11.5)
- moved R79 51.2 mm to (3.75, 3.00), flipped to the bottom, turned to 90 degrees
- moved B1 47.3 mm to (-1.00, -4.50), turned to 270 degrees
- moved R86 45.6 mm to (0.00, -23.0), flipped to the bottom
- moved R81 42.7 mm to (-3.68, -13.6), flipped to the bottom, turned to 270 degrees
- moved R82 30.4 mm to (-2.00, -13.6), flipped to the bottom, turned to 90 degrees
- moved PWR 29.2 mm to (3.75, -24.2), flipped to the bottom, turned to 90 degrees
- moved C5 27.5 mm to (0.00, 3.00), turned to 180 degrees
- moved R77 26.5 mm to (3.75, -26.2), flipped to the bottom
- moved U3 10.0 mm to (0.00, 21.5)
- moved Q1 8.25 mm to (-4.00, -22.0), turned to 270 degrees
- moved LBO 8.25 mm to (-4.00, -24.5), turned to 270 degrees
- moved R83 8.14 mm to (-4.00, -26.2), turned to 0 degrees
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Connections:
- removed net ENABLE: R78.2, U4.11
- net GND: no longer C1.2, C4.2
- net VBAT: now also U4.11; no longer C1.1, C4.1, R78.1
Routing:
- net GND: track 4.26 -> 47.1 mm
- net 5.0V: track 0.00 -> 24.8 mm
- net VBAT: track 0.00 -> 16.3 mm
- net N$73: track 0.00 -> 8.24 mm
- net N$78: track 0.00 -> 6.27 mm
- net N$74: track 0.00 -> 3.71 mm
- net N$75: track 0.00 -> 2.04 mm
- net N$77: track 0.00 -> 1.79 mm
- net N$81: track 0.00 -> 1.70 mm
Other:
- board text added: "PWR"
- board text removed: "2"
- board text removed: "3"

Commit message: dear fucking god
Parts:
- removed PWR: BLUE, microbuilder:CHIPLED_0805_NOOUTLINE
- removed R77: 1K, microbuilder:0805-NO
- moved R79 18.7 mm to (-3.00, -14.4)
- moved R80 17.4 mm to (-4.75, -14.4), turned to 90 degrees
- moved R81 4.53 mm to (-4.75, -18.0)
- moved R82 4.51 mm to (-3.00, -18.0)
- moved R86 4.50 mm to (3.76, -25.5), turned to 180 degrees
- moved LBO 3.85 mm to (-3.76, -20.7)
- moved R83 3.85 mm to (-3.76, -22.4)
- moved Q1 3.44 mm to (-3.92, -25.4)
- moved B1 2.00 mm to (1.00, -4.50), turned to 90 degrees
- moved L1 1.52 mm to (2.44, -20.6)
Connections:
- removed net N$75: PWR.C, R77.1
- net 5.0V: no longer PWR.A
- net GND: no longer R77.2
Routing:
- net GND: track 47.1 -> 32.6 mm
- net VBAT: track 16.3 -> 6.38 mm
- net N$78: track 6.27 -> 0.00 mm
- net N$75: track 2.04 -> 0.00 mm
- net N$81: track 1.70 -> 0.00 mm
- net N$74: track 3.71 -> 2.24 mm
- net 5.0V: track 24.8 -> 23.5 mm
- net N$73: track 8.24 -> 9.31 mm
Other:
- board text removed: "PWR"

Commit message: Remove LBO, change bypass cap
Parts:
- removed C2: 2.2uF, microbuilder:0805-NO
- removed LBO: RED, microbuilder:CHIPLED_0805_NOOUTLINE
- removed Q1: MMUN2133LT1G, transistor:SC59-BEC
- removed R83: 1K, microbuilder:0805-NO
- moved C5 13.2 mm to (-3.36, -9.72)
- moved IC1 6.00 mm to (0.00, 5.50)
- moved B1 1.00 mm to (1.00, -3.50)
- moved R79 0.36 mm to (-3.00, -14.0)
- moved R80 0.36 mm to (-4.75, -14.0)
Connections:
- removed net LBO: Q1.B, U4.12
- removed net N$77: LBO.A, R83.1
- removed net N$78: Q1.C, R83.2
- net 5.0V: no longer C2.1
- net GND: no longer C2.2, LBO.C
- net VBAT: no longer Q1.E
Routing:
- net GND: track 32.6 -> 15.6 mm
- net 5.0V: track 23.5 -> 10.2 mm
- net N$77: track 1.79 -> 0.00 mm

Commit message: holy shit one layer
Parts:
- removed LED3: ORANGE, microbuilder:CHIPLED_0805_NOOUTLINE
- removed LED4: GREEN, microbuilder:CHIPLED_0805_NOOUTLINE
- removed R84: 470, microbuilder:0805-NO
- removed R85: 1K, microbuilder:0805-NO
- moved R81 13.7 mm to (-4.40, -4.28)
- moved R79 13.0 mm to (0.60, -1.52), turned to 180 degrees
- moved R80 12.6 mm to (-2.96, -1.53), turned to 180 degrees
- moved C5 11.7 mm to (0.00, 1.50)
- moved R82 10.5 mm to (-4.40, -7.64), turned to 270 degrees
- moved B1 10.3 mm to (-0.96, -13.6), turned to 270 degrees
- moved U4 7.44 mm to (-0.04, -6.09)
- moved R86 4.66 mm to (0.04, -28.3), turned to 0 degrees
- moved IC1 2.50 mm to (0.00, 8.00)
- moved L1 2.44 mm to (0.00, -20.8)
- moved J2 0.56 mm to (0.00, -34.6)
- moved C6 0.48 mm to (0.00, -29.9)
- moved U5 0.44 mm to (0.00, -25.6), turned to 90 degrees
Connections:
- removed net N$79: LED3.C, R84.1
- removed net N$80: R84.2, R85.2, U5.1
- removed net N$82: LED4.A, R85.1
- net GND: no longer LED4.C
- net VDD1: no longer LED3.A
Routing:
- net GND: track 15.6 -> 84.5 mm
- net VBAT: track 6.38 -> 49.9 mm
- net 5.0V: track 10.2 -> 29.3 mm
- net N$73: track 9.31 -> 21.7 mm
- net VDD1: track 4.43 -> 10.3 mm
- net N$76: track 0.00 -> 4.13 mm
- net N$82: track 1.92 -> 0.00 mm
- net N$79: track 1.92 -> 0.00 mm
- net N$81: track 0.00 -> 1.90 mm
- net N$74: track 2.24 -> 3.86 mm
Other:
- board text added: "+"
- board text removed: "CHRG"
- board text removed: "DONE"
- board text removed: "LOW"

Commit message: micro
Parts:
- removed U3: ATSAMD21G-A, SparkFun-IC-Microcontroller:TQFP-48
- added C1: 1uF, microbuilder:0805-NO
- added C2: 0.1uF, microbuilder:0805-NO
- added C3, C4: 10pF, rcl:C0805
- added MCU: ATSAMD21E, adafruit:TQFP32-08
- added Y1: 32.768kHz, SparkFun-Clocks:CRYSTAL-SMD-3.2X1.5MM
Connections:
- new net D+: J2.D+, MCU.24
- new net D-: J2.D-, MCU.23
- new net N$75: C1.2, MCU.29
- new net N$77: C2.2, MCU.30, MCU.9
- new net N$78: C4.1, MCU.2, Y1.P$1
- new net N$79: C3.1, MCU.1, Y1.P$2
- new net RESET: MCU.26
- new net SWCLK: MCU.31
- new net SWDIO: MCU.32
- net 3V3: now also C1.1, C2.1
- net GND: now also C3.2, C4.2, MCU.10, MCU.28
Routing:
- net D-: track 0.00 -> 53.5 mm
- net D+: track 0.00 -> 53.3 mm
- net GND: track 84.5 -> 87.0 mm

Commit message: diff pair
Parts:
- moved C1 10.4 mm to (4.00, 23.5)
- moved C2 8.00 mm to (7.68, 18.8)
- renumbered MCU to U3
Connections:
- net D+ renamed USB_P
- net D- renamed USB_N
Routing:
- net USB_N: track 53.5 -> 60.6 mm
- net USB_P: track 53.3 -> 59.9 mm
- net N$79: track 0.00 -> 6.25 mm
- net N$78: track 0.00 -> 5.48 mm
