File: LEDboard.brd (EAGLE design)
At the start: 72 x 72 mm, 322 parts, among them J1 JTAG, U1 IS31FL3741_QFN60, U2 IS31FL3741_QFN60, U3 ATSAMD21E, U4 TPS61090RSAR, U5 MCP73831T-2ACI/OT, Y1 32.768kHz

Commit message: update
Routing:
- net U2SW8: track 157.3 -> 294.7 mm, vias 8 -> 9
- net U2SW2: track 131.4 -> 234.3 mm, vias 12 -> 14
- net U2SW6: track 110.2 -> 143.4 mm, vias 9 -> 12
- net U1SW1: track 135.6 -> 168.4 mm, vias 9 -> 12
- net U2SW1: track 156.0 -> 184.2 mm, vias 11 -> 15
- net U2SW3: track 139.6 -> 167.7 mm, vias 10 -> 14
- net U1SW8: track 103.0 -> 126.1 mm, vias 8 -> 9
- net N$197: track 77.8 -> 55.3 mm
- net U2SW4: track 119.3 -> 140.6 mm, vias 10 -> 14
- net N$140: track 28.0 -> 6.99 mm
- net N$130: track 24.5 -> 3.66 mm
- net U2SW5: track 115.8 -> 131.6 mm, vias 9 -> 12
- net U1SW2: track 134.2 -> 148.3 mm, vias 11 -> 14
- net N$95: track 28.0 -> 14.8 mm
- net N$306: track 13.1 -> 0.00 mm
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
Commit message: routing
Routing:
- net U2SW2: track 234.3 -> 281.2 mm, vias 14 -> 18
- net U1SW1: track 168.4 -> 199.9 mm, vias 12 -> 17
- net U2SW3: track 167.7 -> 199.0 mm, vias 14 -> 17
- net N$131: track 28.0 -> 0.00 mm
- net N$133: track 28.0 -> 0.00 mm
- net U1SW3: track 159.5 -> 184.4 mm, vias 12 -> 17
- net U2SW8: track 294.7 -> 319.2 mm, vias 9 -> 12
- net U2SW7: track 112.7 -> 136.5 mm, vias 10 -> 15
- net N$195: track 57.3 -> 35.6 mm
- net N$127: track 28.0 -> 6.99 mm
- net N$100: track 19.2 -> 0.00 mm
- net U1SW4: track 130.1 -> 147.6 mm, vias 11 -> 16
- net N$160: track 19.8 -> 2.45 mm
- net U1SW5: track 134.0 -> 150.9 mm, vias 9 -> 13
- net U1SW2: track 148.3 -> 164.6 mm, vias 14 -> 16
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
Commit message: another ring
Routing:
- net U1SW2: track 164.6 -> 195.2 mm, vias 16 -> 19
- net U1SW3: track 184.4 -> 213.8 mm, vias 17 -> 19
- net N$107: track 28.0 -> 0.00 mm
- net N$109: track 28.0 -> 0.00 mm
- net N$185: track 41.4 -> 20.0 mm
- net U1SW8: track 137.2 -> 157.9 mm, vias 13 -> 14
- net N$114: track 17.5 -> 0.00 mm
- net N$100: track 0.00 -> 16.1 mm
- net N$241: track 13.1 -> 0.00 mm
- net U1SW4: track 147.6 -> 159.9 mm, vias 16 -> 18
- net U1SW5: track 150.9 -> 162.1 mm, vias 13 -> 15
- net N$196: track 10.6 -> 0.00 mm
- net N$102: track 10.6 -> 0.00 mm
- net U1SW6: track 123.3 -> 133.3 mm, vias 11 -> 14
- net U1SW7: track 127.5 -> 135.7 mm, vias 12 -> 14
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
Commit message: difficulty
Routing:
- net U2SW5: track 143.1 -> 185.1 mm, vias 14 -> 17
- net N$124: track 28.0 -> 0.00 mm
- net N$122: track 28.0 -> 0.00 mm
- net U2SW6: track 151.9 -> 177.7 mm, vias 14 -> 16
- net U2SW8: track 319.2 -> 341.9 mm, vias 12 -> 15
- net U2SW4: track 153.4 -> 174.2 mm, vias 16 -> 18
- net N$173: track 19.7 -> 0.00 mm
- net N$120: track 14.0 -> 0.00 mm
- net N$217: track 40.2 -> 30.7 mm
- net U1SW8: track 157.9 -> 165.9 mm, vias 14 -> 15
- net N$75: track 5.24 -> 0.00 mm
- net U1CS15: track 38.6 -> 42.4 mm
- net U2CS15: track 40.1 -> 42.5 mm
- net USB_P: track 72.3 -> 70.2 mm
- net USB_N: track 57.7 -> 55.9 mm
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
Commit message: another row
Routing:
- net U1SW5: track 162.1 -> 201.8 mm, vias 15 -> 20
- net 5.0V: track 80.7 -> 54.9 mm
- net U2SW3: track 199.0 -> 223.4 mm, vias 17 -> 19
- net U1SW3: track 213.8 -> 236.8 mm, vias 19 -> 20
- net N$144: track 19.9 -> 0.00 mm
- net N$184: track 19.8 -> 0.00 mm
- net N$193: track 51.9 -> 32.8 mm
- net N$142: track 17.5 -> 0.00 mm
- net U2SW5: track 185.1 -> 202.1 mm, vias 17 -> 19
- net U1SW4: track 159.9 -> 176.7 mm, vias 18 -> 20
- net N$186: track 16.6 -> 0.00 mm
- net N$163: track 16.6 -> 0.00 mm
- net U1SW6: track 133.3 -> 149.2 mm, vias 14 -> 16
- net N$75: track 0.00 -> 14.7 mm
- net N$93: track 19.2 -> 5.24 mm
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
Commit message: begin removal
Routing:
- net U1SW9: track 131.7 -> 12.8 mm, vias 12 -> 0
- net N$287: track 73.1 -> 0.00 mm
- net U2SW8: track 341.9 -> 271.6 mm
- net N$214: track 67.5 -> 0.00 mm
- net N$183: track 61.9 -> 0.00 mm
- net N$289: track 61.9 -> 0.30 mm
- net N$164: track 59.2 -> 0.00 mm
- net N$215: track 59.1 -> 0.00 mm
- net N$208: track 58.1 -> 0.00 mm
- net N$197: track 55.3 -> 0.00 mm
- net N$216: track 53.6 -> 0.00 mm
- net N$209: track 45.1 -> 0.00 mm
- net U2SW6: track 177.7 -> 220.0 mm, vias 16 -> 18
- net N$195: track 35.6 -> 0.00 mm
- net N$193: track 32.8 -> 0.00 mm
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