File: LEDboard.brd (EAGLE design)
At the start: 72 x 72 mm, 322 parts, among them J1 JTAG, U1 IS31FL3741_QFN60, U2 IS31FL3741_QFN60, U3 ATSAMD21E, U4 TPS61090RSAR, U5 MCP73831T-2ACI/OT, Y1 32.768kHz

Commit message: fuckall
Routing:
- net U1CS30: track 40.7 -> 65.0 mm, vias 0 -> 4
- net U1CS29: track 39.6 -> 56.1 mm, vias 0 -> 3
- net N$147: track 19.9 -> 11.7 mm
- net N$273: track 13.1 -> 4.90 mm
- net U1CS28: track 39.5 -> 47.1 mm, vias 0 -> 3
- net N$101: track 10.5 -> 6.99 mm

Commit message: more rows
Routing:
- net U1CS20: track 44.9 -> 67.4 mm, vias 2 -> 6
- net U1CS19: track 38.8 -> 60.5 mm, vias 2 -> 6
- net N$153: track 19.9 -> 0.00 mm
- net U1CS21: track 46.7 -> 66.2 mm, vias 2 -> 5
- net N$281: track 13.1 -> 0.00 mm
- net U1CS16: track 39.2 -> 52.3 mm, vias 0 -> 2
- net U1CS18: track 42.6 -> 54.2 mm, vias 0 -> 2
- net U1CS17: track 40.5 -> 52.0 mm, vias 0 -> 2
- net U1CS25: track 55.3 -> 65.8 mm, vias 2 -> 5
- net U1CS22: track 39.2 -> 47.8 mm, vias 0 -> 2
- net U1CS23: track 40.7 -> 48.5 mm, vias 0 -> 2
- net N$282: track 6.99 -> 0.00 mm
- net N$292: track 6.53 -> 0.00 mm
- net U1CS24: track 41.2 -> 47.7 mm, vias 0 -> 2
- net U1CS26: track 41.3 -> 47.1 mm, vias 2 -> 3
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
Commit message: another bunch
Routing:
- net U1CS14: track 38.8 -> 90.0 mm, vias 2 -> 6
- net U1CS15: track 42.4 -> 92.4 mm, vias 2 -> 6
- net U1CS13: track 38.8 -> 79.0 mm, vias 2 -> 4
- net N$155: track 19.9 -> 0.00 mm
- net N$192: track 17.0 -> 0.00 mm
- net N$147: track 11.7 -> 0.00 mm
- net N$101: track 6.99 -> 0.00 mm
- net U1SW9: track 132.5 -> 129.5 mm
- net N$92: track 0.00 -> 2.45 mm
- net N$87: track 2.45 -> 0.00 mm
- net N$148: track 1.63 -> 0.00 mm
- net U1CS34: track 81.2 -> 82.4 mm

Commit message: finished left hand
Routing:
- net U1CS8: track 35.5 -> 82.3 mm, vias 2 -> 6
- net U1CS9: track 56.8 -> 95.8 mm, vias 2 -> 5
- net U1CS7: track 33.7 -> 72.1 mm, vias 2 -> 6
- net U1CS4: track 18.4 -> 45.5 mm, vias 0 -> 2
- net U1CS5: track 24.6 -> 51.5 mm, vias 0 -> 2
- net U1CS6: track 27.6 -> 51.8 mm, vias 0 -> 2
- net U1CS10: track 36.8 -> 53.4 mm, vias 2 -> 3
- net U1CS11: track 53.1 -> 69.4 mm, vias 2 -> 4
- net U1CS13: track 79.0 -> 93.9 mm, vias 4 -> 6
- net U1CS12: track 39.3 -> 53.9 mm, vias 2 -> 4
- net N$286: track 13.1 -> 0.00 mm
- net N$236: track 13.1 -> 0.00 mm
- net N$235: track 13.1 -> 0.00 mm
- net N$234: track 13.1 -> 0.00 mm
- net VBAT: track 44.5 -> 40.7 mm
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
Commit message: omg jesus christ
Routing:
- net U2CS33: track 39.7 -> 106.9 mm, vias 2 -> 6
- net U2CS36: track 39.9 -> 104.1 mm, vias 0 -> 4
- net U2CS32: track 39.5 -> 100.3 mm, vias 2 -> 6
- net U2CS31: track 38.3 -> 94.3 mm, vias 2 -> 5
- net U2CS7: track 34.4 -> 82.5 mm, vias 2 -> 6
- net U2CS14: track 38.1 -> 84.9 mm, vias 2 -> 6
- net U2CS13: track 38.1 -> 82.8 mm, vias 2 -> 6
- net U2CS8: track 36.6 -> 80.2 mm, vias 2 -> 6
- net U2CS9: track 38.9 -> 82.0 mm, vias 2 -> 6
- net U2CS25: track 38.9 -> 79.7 mm, vias 2 -> 5
- net U2CS4: track 21.5 -> 60.7 mm, vias 2 -> 5
- net U2CS35: track 39.6 -> 78.0 mm, vias 0 -> 4
- net U2CS15: track 42.5 -> 80.2 mm, vias 2 -> 6
- net U2CS26: track 41.9 -> 77.7 mm, vias 2 -> 5
- net U2CS27: track 40.3 -> 75.6 mm, vias 2 -> 6
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
Commit message: Beginning the final routing
Routing:
- net U2SW7: track 181.6 -> 200.0 mm, vias 21 -> 23
- net U2SW5: track 200.1 -> 216.2 mm, vias 22 -> 23
- net U1SW4: track 193.5 -> 209.1 mm, vias 25 -> 27
- net U1SW6: track 196.6 -> 210.0 mm, vias 22 -> 24
- net U2SW6: track 218.9 -> 232.1 mm, vias 18 -> 21
- net U2SW4: track 178.2 -> 190.9 mm, vias 20 -> 22
- net U1SW8: track 157.4 -> 167.6 mm, vias 21 -> 23
- net U1SW9: track 129.4 -> 138.7 mm, vias 16 -> 17
- net U1SW7: track 178.7 -> 187.7 mm, vias 22 -> 24
- net U2SW8: track 281.8 -> 290.5 mm, vias 18 -> 21
- net U2SW2: track 257.1 -> 265.0 mm
- net U1SW2: track 227.5 -> 233.8 mm
- net N$229: track 4.90 -> 0.00 mm
- net N$258: track 4.90 -> 0.00 mm
- net U2SW9: track 111.2 -> 115.9 mm, vias 13 -> 15
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
Commit message: one side done
Parts:
- removed R77: 0 Ohm, SparkFun-Resistors:1206
- moved C16 0.51 mm to (16.1, 12.6)
- moved C9 0.43 mm to (-16.0, -12.5)
Connections:
- net 5.0V: no longer R77.1, R77.2
Routing:
- net N$1: track 0.00 -> 50.4 mm
- net N$2: track 0.00 -> 48.7 mm
- net N$3: track 0.00 -> 47.4 mm
- net N$4: track 0.00 -> 44.5 mm
- net N$5: track 0.00 -> 42.2 mm
- net N$6: track 0.00 -> 40.6 mm
- net 5.0V: track 37.0 -> 70.4 mm
- net N$47: track 0.00 -> 32.0 mm
- net N$60: track 0.66 -> 31.4 mm
- net N$58: track 0.00 -> 30.0 mm
- net N$48: track 0.00 -> 29.8 mm
- net N$59: track 0.00 -> 29.6 mm
- net N$54: track 0.00 -> 29.3 mm
- net N$7: track 0.00 -> 29.0 mm
- net N$53: track 0.00 -> 28.3 mm
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
Commit message: complete
Parts:
- moved C16 4.83 mm to (12.0, 10.1), turned to 0 degrees
Routing:
- net N$13: track 0.00 -> 40.6 mm
- net N$14: track 0.00 -> 40.1 mm
- net N$20: track 0.00 -> 39.9 mm
- net N$15: track 0.00 -> 39.3 mm
- net N$19: track 0.00 -> 39.1 mm
- net N$72: track 0.00 -> 38.5 mm
- net N$71: track 0.00 -> 37.1 mm
- net N$21: track 0.00 -> 36.8 mm
- net N$70: track 0.00 -> 36.2 mm
- net N$69: track 0.00 -> 35.7 mm
- net N$68: track 0.00 -> 34.7 mm
- net N$26: track 0.00 -> 34.3 mm
- net N$67: track 0.00 -> 34.3 mm
- net N$66: track 0.00 -> 33.3 mm
- net N$65: track 0.00 -> 33.1 mm
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