File: LEDboard.sch (EAGLE design)
At the start: 323 parts, among them J1 JTAG, U1 IS31FL3741_QFN60, U2 IS31FL3741_QFN60, U3 ATSAMD21E, U4 TPS61090RSAR, U5 MCP73831T-2ACI/OT, Y1 32.768kHz

Commit message: I think I fucked something up
Parts:
- removed R83, R84: 0 Ohm, SparkFun-Resistors:RESISTOR1206
Connections:
- removed net N$75: R83.1, U3.PA22
- removed net N$77: R84.1, U3.PA23
- net SCL: now also U3.PA23; no longer R84.2
- net SDA: now also U3.PA22; no longer R83.2
Changed lines of the file:
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@@
 <part name="U$17" library="microbuilder" deviceset="GND" device=""/>
 <part name="U$18" library="microbuilder" deviceset="GND" device=""/>
-<part name="R83" library="SparkFun-Resistors" library_urn="urn:adsk.eagle:library:532" deviceset="RESISTOR" device="1206" package3d_urn="urn:adsk.eagle:package:39654/1" value="0 Ohm"/>
-<part name="R84" library="SparkFun-Resistors" library_urn="urn:adsk.eagle:library:532" deviceset="RESISTOR" device="1206" package3d_urn="urn:adsk.eagle:package:39654/1" value="0 Ohm"/>
 <part name="U$20" library="TindieBadge" deviceset="ALPSSLIDESW" device="" value="TINDIE_SWITCH"/>
 <part name="U$21" library="microbuilder" deviceset="GND" device=""/>
@@
 <attribute name="VALUE" x="101.6" y="24.13" size="1.778" layer="96"/>
 </instance>
-<instance part="R83" gate="G$1" x="76.2" y="22.86" smashed="yes">
-<attribute name="NAME" x="76.2" y="24.384" size="1.778" layer="95" font="vector" align="bottom-center"/>
-<attribute name="VALUE" x="76.2" y="21.336" size="1.778" layer="96" font="vector" align="top-center"/>
-</instance>
-<instance part="R84" gate="G$1" x="76.2" y="20.32" smashed="yes">
-<attribute name="NAME" x="76.2" y="21.844" size="1.778" layer="95" font="vector" align="bottom-center"/>
-<attribute name="VALUE" x="76.2" y="18.796" size="1.778" layer="96" font="vector" align="top-center"/>
-</instance>
 <instance part="R87" gate="G$1" x="96.52" y="35.56" smashed="yes" rot="R90">
 <attribute name="NAME" x="93.98" y="35.56" size="1.27" layer="95" font="vector" rot="R90" align="center"/>
@@
 <segment>
 <wire x1="86.36" y1="22.86" x2="81.28" y2="22.86" width="0.1524" layer="91"/>
-<pinref part="R83" gate="G$1" pin="2"/>
+<pinref part="U3" gate="G$1" pin="PA22"/>
+<wire x1="63.5" y1="22.86" x2="71.12" y2="22.86" width="0.1524" layer="91"/>
+<wire x1="81.28" y1="22.86" x2="71.12" y2="22.86" width="0.1524" layer="91"/>
 </segment>
 </net>
@@
 <segment>
 <wire x1="86.36" y1="20.32" x2="81.28" y2="20.32" width="0.1524" layer="91"/>
-<pinref part="R84" gate="G$1" pin="2"/>
-</segment>
-</net>
-<net name="N$75" class="0">
-<segment>
-<pinref part="U3" gate="G$1" pin="PA22"/>
-<pinref part="R83" gate="G$1" pin="1"/>
-<wire x1="63.5" y1="22.86" x2="71.12" y2="22.86" width="0.1524" layer="91"/>
-</segment>
-</net>
-<net name="N$77" class="0">
-<segment>
 <pinref part="U3" gate="G$1" pin="PA23"/>
-<pinref part="R84" gate="G$1" pin="1"/>
 <wire x1="63.5" y1="20.32" x2="71.12" y2="20.32" width="0.1524" layer="91"/>
+<wire x1="71.12" y1="20.32" x2="81.28" y2="20.32" width="0.1524" layer="91"/>
 </segment>
 </net>
