File: LEDboard.sch (EAGLE design)
At the start: 321 parts, among them J1 JTAG, U1 IS31FL3741_QFN60, U2 IS31FL3741_QFN60, U3 ATSAMD21E, U4 TPS61090RSAR, U5 MCP73831T-2ACI/OT, Y1 32.768kHz

Commit message: Fixed address pins
Connections:
- net 3V3: now also U2.ADDR
- net GND: no longer U2.ADDR
Other:
- note added: "ADDR connect to ground ADDR=00 See pg. 7 of datasheet"
- note added: "ADDR connects to vcc ADDR = 11 See pg. 7 of datasheet"
- note removed: "Fix the address things"
Changed lines of the file:
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@@
 <part name="R83" library="microbuilder" deviceset="RESISTOR" device="0805_NOOUTLINE" value="200K"/>
 <part name="U$25" library="microbuilder" deviceset="5.0V" device="" value="3V3"/>
+<part name="+3V3" library="supply1" library_urn="urn:adsk.eagle:library:371" deviceset="+3V3" device=""/>
 </parts>
 <sheets>
@@
 <text x="76.2" y="342.9" size="6.4516" layer="91">change these to cree
 UHD1110-FKA LEDs</text>
+<text x="208.28" y="261.62" size="1.778" layer="97">ADDR connect to ground
+ADDR=00
+See pg. 7 of datasheet</text>
 </plain>
 <instances>
@@
 <wire x1="165.1" y1="-101.6" x2="170.18" y2="-101.6" width="0.1524" layer="94"/>
 <wire x1="170.18" y1="-101.6" x2="167.64" y2="-99.06" width="0.1524" layer="94"/>
-<text x="-129.54" y="241.3" size="19.05" layer="94">LED Array Right</text>
-<text x="-5.08" y="139.7" size="5.08" layer="91">Fix the address things</text>
+<text x="-121.92" y="246.38" size="19.05" layer="94">LED Array Right</text>
+<text x="45.72" y="134.62" size="1.778" layer="97">ADDR connects to vcc
+ADDR = 11
+See pg. 7 of datasheet</text>
 </plain>
 <instances>
@@
 <attribute name="VALUE" x="53.34" y="167.64" size="1.778" layer="96" rot="R90"/>
 </instance>
+<instance part="+3V3" gate="G$1" x="63.5" y="132.08" smashed="yes">
+<attribute name="VALUE" x="60.96" y="127" size="1.778" layer="96" rot="R90"/>
+</instance>
 </instances>
 <busses>
@@
 <pinref part="GND1" gate="1" pin="GND"/>
 <wire x1="60.96" y1="106.68" x2="60.96" y2="91.44" width="0.1524" layer="91"/>
-<wire x1="68.58" y1="119.38" x2="60.96" y2="119.38" width="0.1524" layer="91"/>
-<wire x1="60.96" y1="119.38" x2="60.96" y2="106.68" width="0.1524" layer="91"/>
 <junction x="60.96" y="106.68"/>
 <pinref part="R75" gate="G$1" pin="1"/>
 <wire x1="53.34" y1="111.76" x2="53.34" y2="106.68" width="0.1524" layer="91"/>
 <wire x1="53.34" y1="106.68" x2="60.96" y2="106.68" width="0.1524" layer="91"/>
-<pinref part="U2" gate="G$1" pin="ADDR"/>
 <pinref part="U2" gate="G$1" pin="GND"/>
 </segment>
@@
 <pinref part="R76" gate="G$1" pin="2"/>
 </segment>
+<segment>
+<pinref part="+3V3" gate="G$1" pin="+3V3"/>
+<wire x1="63.5" y1="127" x2="63.5" y2="129.54" width="0.1524" layer="91"/>
+<pinref part="U2" gate="G$1" pin="ADDR"/>
+<wire x1="68.58" y1="119.38" x2="63.5" y2="119.38" width="0.1524" layer="91"/>
+<wire x1="63.5" y1="119.38" x2="63.5" y2="127" width="0.1524" layer="91"/>
+</segment>
 </net>

Commit message: Fixed tiny issue, now works
Connections:
- new net N$77: U3.VCORE
- net 3V3: no longer U3.VCORE
Changed lines of the file:
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@@
 <wire x1="22.86" y1="73.66" x2="22.86" y2="78.74" width="0.1524" layer="91"/>
 <wire x1="22.86" y1="71.12" x2="22.86" y2="73.66" width="0.1524" layer="91"/>
-<wire x1="22.86" y1="66.04" x2="22.86" y2="71.12" width="0.1524" layer="91"/>
 <wire x1="25.4" y1="71.12" x2="22.86" y2="71.12" width="0.1524" layer="91"/>
-<junction x="22.86" y="71.12"/>
 <pinref part="U3" gate="G$1" pin="VDD"/>
 <wire x1="25.4" y1="71.12" x2="33.02" y2="71.12" width="0.1524" layer="91"/>
-<pinref part="U3" gate="G$1" pin="VCORE"/>
-<wire x1="33.02" y1="66.04" x2="30.48" y2="66.04" width="0.1524" layer="91"/>
-<wire x1="22.86" y1="66.04" x2="30.48" y2="66.04" width="0.1524" layer="91"/>
 </segment>
 <segment>
@@
 </segment>
 </net>
+<net name="N$77" class="0">
+<segment>
+<pinref part="U3" gate="G$1" pin="VCORE"/>
+<wire x1="33.02" y1="66.04" x2="30.48" y2="66.04" width="0.1524" layer="91"/>
+</segment>
+</net>
